Commit message: Parte11

File: Parte11/psr_parte11_scara/urdf/scara.urdf (robot description, URDF)
Before this commit: robot myscara, 2 links, 1 joints
Links:
- added link link1b; visual cylinder length=0.6 radius=0.3
- added link link2; visual box size=3 0.6 0.6
- added link link2b; visual cylinder length=0.6 radius=0.3
- added link link3; visual cylinder length=3 radius=0.15
Joints:
- added joint link1_to_link1b: type fixed, parent link1, child link1b, origin xyz=0 0 -0.3 rpy=0 0 0
- added joint link1_to_link2: type revolute, parent link1, child link2, origin xyz=3 0 0 rpy=0 0 0, axis 0 0 1, limit lower=-3.14 upper=3.14 effort=1000.0 velocity=0.5
- added joint link2_to_link2b: type fixed, parent link2, child link2b, origin xyz=0 0 -0.3 rpy=0 0 0
- added joint link2_to_link3: type prismatic, parent link2, child link3, origin xyz=3 0 0 rpy=0 0 0, axis 0 0 -1, limit lower=-1.5 upper=1.5 effort=1000.0 velocity=0.5
