Commit message: Parte12

File: Parte12/p_rferreira_description/urdf/p_rferreira.gazebo.xacro (robot description, xacro)
@@ -6,5 +6,5 @@
   <gazebo reference="base_link">
 <!--    <material>Gazebo/DarkGrey</material>-->
-      <material>Gazebo/Yellow</material>
+      <material>Gazebo/${player_color}</material>
   </gazebo>
   <gazebo reference="wheel_left_link">

File: Parte12/p_rferreira_description/urdf/p_rferreira.urdf.xacro (robot description, xacro)
@@ -1,5 +1,14 @@
 <?xml version="1.0" ?>
-<robot name="turtlebot3_waffle_pi" xmlns:xacro="http://ros.org/wiki/xacro">
-  <xacro:include filename="$(find turtlebot3_description)/urdf/common_properties.xacro"/>
+<robot name="team_hunt_player" xmlns:xacro="http://ros.org/wiki/xacro">
+<!--  Argument-->
+  <xacro:arg name="player_name" default="p_rferreira"/>
+  <xacro:arg name="player_color" default="Red"/>
+<!--  copy property -->
+<!--  properties are used as ${property}-->
+  <xacro:property name="player_name" value="$(arg player_name)"/>
+  <xacro:property name="player_color" value="$(arg player_color)"/>
+<!--  Includes-->
+<!--  <xacro:include filename="$(find turtlebot3_description)/urdf/common_properties.xacro"/>-->
+  <xacro:include filename="$(find p_rferreira_description)/urdf/properties.xacro"/>
 <!--  <xacro:include filename="$(find turtlebot3_description)/urdf/turtlebot3_waffle_pi.gazebo.xacro"/>-->
   <xacro:include filename="$(find p_rferreira_description)/urdf/p_rferreira.gazebo.xacro"/>
@@ -16,5 +25,6 @@
         <mesh filename="package://turtlebot3_description/meshes/bases/waffle_pi_base.stl" scale="0.001 0.001 0.001"/>
       </geometry>
-      <material name="light_black"/>
+<!--      <material name="light_black"/>-->
+      <material name="$(arg player_color)"/>
     </visual>
     <collision>
